File: gmm7550.kicad/connectors.kicad_sch (KiCad schematic)
At the start: 9 parts, among them P1 10144518-061802LF, P2 10144518-061802LF, P3 10144518-061802LF, P4 10144518-061802LF, P5 10144518-061802LF

Commit message: Update copyright years and increment revision
Other:
- note added: "Copyright (c) 2020-2022 Anton Kuzmin Licensed under CERN-OHL-P v2 https://github.com/gmm-7550/"
- note removed: "Copyright (c) 2020-2022 Anton Kuzmin Licensed under CERN-OHL-P v2 https://github.com/ak-fau/gmm7550.git"
Changed lines of the file:
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@@
   (title_block
     (title "GateMate FPGA Module: GMM-7550")
-    (date "2022-04-24")
-    (rev "2.1")
+    (date "2022-04-27")
+    (rev "2.2")
   )
   (junction (at 106.68 82.55) (diameter 0) (color 0 0 0 0)
@@
     (stroke (width 0) (type default))
   )
-  (text "Copyright (c) 2020-2022  Anton Kuzmin\nLicensed under CERN-OHL-P v2\nhttps://github.com/ak-fau/gmm7550.git"
+  (text "Copyright (c) 2020-2022  Anton Kuzmin\nLicensed under CERN-OHL-P v2\nhttps://github.com/gmm-7550/"
     (at 198.12 179.07 0)
     (effects (font (size 2.54 2.54)) (justify left bottom))
