File: gmm7550.kicad/io.kicad_sch (KiCad schematic)
At the start: 49 parts, among them U1 CCGM1A1

Commit message: Update copyright years and increment revision
Other:
- note added: "Copyright (c) 2020-2024 Anton Kuzmin Licensed under CERN-OHL-P v2 https://github.com/gmm-7550/"
- note removed: "Copyright (c) 2020-2022 Anton Kuzmin Licensed under CERN-OHL-P v2 https://github.com/ak-fau/gmm7550.git"
Changed lines of the file:
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@@
   (title_block
     (title "GateMate FPGA Module: GMM-7550")
-    (date "2022-04-24")
-    (rev "2.1")
+    (date "2022-04-27")
+    (rev "2.2")
   )
   (junction (at 33.02 109.22) (diameter 0) (color 0 0 0 0)
@@
     (stroke (width 0) (type default))
   )
-  (text "Copyright (c) 2020-2022  Anton Kuzmin\nLicensed under CERN-OHL-P v2\nhttps://github.com/ak-fau/gmm7550.git"
+  (text "Copyright (c) 2020-2024  Anton Kuzmin\nLicensed under CERN-OHL-P v2\nhttps://github.com/gmm-7550/"
     (at 198.12 179.07 0)
     (effects (font (size 2.54 2.54)) (justify left bottom))
