File: hat-gmm7550.kicad/hat-gmm7550.kicad_pcb (KiCad board)
At the start: 4 copper layers, 65 x 56 mm, 83 parts, among them J1 VisionFive_GPIO, J10 Pmod 2x6, J2 Conn_01x02, J3 Conn_02x02_Odd_Even, J4 DNI, J5 DNI, J6 10144517-064802LF, J7 10144517-064802LF, J8 JTAG, J9 Pmod 2x6, Q1 NX6008NBK, Q2 NX6008NBK, Q3 NX6008NBK, Q4 FDC855N, U1 CAT24C32Y, U2 74LVC1G07, U3 ADM1177, U4 LSF0204PW, U5 LSF0204PW, U6 LSF0204PW, U7 LSF0204PW, U8 LSF0204PW, U9 LSF0204PW

Commit message: Update copyright years and increment revision
Other:
- board text added: "rev 1.2"
- board text removed: "rev 1.1"
Changed lines of the file:
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@@
     (effects (font (size 1.5 1.5) (thickness 0.15)))
   )
-  (gr_text "rev 1.1" (at 130.2 58) (layer "F.SilkS")
+  (gr_text "rev 1.2" (at 130.2 58) (layer "F.SilkS")
     (effects (font (size 1.5 1.5) (thickness 0.15)))
   )
