File: usb3-gmm7550.kicad/gmm-7550.kicad_sch (KiCad schematic)
At the start: 36 parts, among them J5 10144517-061802LF, Q1 NX6008NBK, Q2 NX6008NBK, Q3 NX6008NBK, SW1 SW_Push, U10 74LVC1G07, U11 INA180A2, U9 SiP32510

Commit message: Final touches -- revision 1.0 schematic is released
Parts:
- U10: value 74LVC1G07 -> SN74LVC1G07DBV
Changed lines of the file:
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@@
 	(title_block
 		(title "GMM-7550 USB3 Adapter")
-		(date "2025-10-01")
-		(rev "0.9.5")
+		(date "2025-10-10")
+		(rev "1.0")
 	)
 	(text "5.0V --> 2.27V\n5.5V --> 2.5V"
@@
 			)
 		)
-		(property "Value" "74LVC1G07"
-			(at 114.3 58.42 0)
+		(property "Value" "SN74LVC1G07DBV"
+			(at 118.11 58.42 0)
 			(effects
 				(font
