File: usb3-gmm7550.kicad/usb3-pd.kicad_sch (KiCad schematic)
At the start: 29 parts, among them J6 DNI, Q4 NX6008NBK, U18 FUSB303BTMX, U19 SiP32508DT, U20 LM66200DRLR, U21 74LVC1G06

Commit message: Layout WIP: split power plane (internal layer 2)
Parts:
- added C53: 1.0uF, Capacitor_SMD:C_0402_1005Metric, symbol Device:C_Small
Connections:
- net +5V: now also C53.1
- net GND: now also C53.2
- net PD_DIS renamed PD_DISCH
Changed lines of the file:
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@@
 	)
 	(junction
+		(at 71.12 43.18)
+		(diameter 0)
+		(color 0 0 0 0)
+	)
+	(junction
 		(at 220.98 48.26)
 		(diameter 0)
@@
 	)
 	(junction
+		(at 76.2 71.12)
+		(diameter 0)
+		(color 0 0 0 0)
+	)
+	(junction
 		(at 101.6 57.15)
 		(diameter 0)
@@
 	(wire
 		(pts
-			(xy 76.2 71.12) (xy 90.17 71.12)
-		)
-		(stroke
-			(width 0)
-			(type default)
-		)
-	)
-	(wire
-		(pts
 			(xy 128.27 100.33) (xy 128.27 101.6)
 		)
@@
 	(wire
 		(pts
+			(xy 71.12 54.61) (xy 71.12 71.12)
+		)
+		(stroke
+			(width 0)
+			(type default)
+		)
+	)
+	(wire
+		(pts
 			(xy 132.08 111.76) (xy 132.08 101.6)
 		)
@@
 	(wire
 		(pts
+			(xy 76.2 71.12) (xy 90.17 71.12)
+		)
+		(stroke
+			(width 0)
+			(type default)
+		)
+	)
+	(wire
+		(pts
 			(xy 128.27 119.38) (xy 142.24 119.38)
 		)
@@
 	(wire
 		(pts
+			(xy 71.12 43.18) (xy 71.12 49.53)
+		)
+		(stroke
+			(width 0)
+			(type default)
+		)
+	)
+	(wire
+		(pts
 			(xy 114.3 43.18) (xy 114.3 49.53)
 		)
@@
 	(wire
 		(pts
+			(xy 71.12 71.12) (xy 76.2 71.12)
+		)
+		(stroke
+			(width 0)
+			(type default)
+		)
+	)
+	(wire
+		(pts
 			(xy 66.04 124.46) (xy 92.71 124.46)
 		)
@@
 		)
 	)
-	(global_label "PD_DIS"
+	(global_label "PD_DISCH"
 		(shape input)
 		(at 66.04 63.5 180)
@@
 		)
 		(property "Intersheetrefs" "${INTERSHEET_REFS}"
-			(at 56.4629 63.5 0)
+			(at 53.8624 63.5 0)
 			(effects
 				(font
@@
 					(unit 1)
 				)
+			)
+		)
+	)
+	(symbol
+		(lib_id "Device:C_Small")
+		(at 71.12 52.07 0)
+		(unit 1)
+		(exclude_from_sim no)
+		(in_bom yes)
+		(on_board yes)
+		(dnp no)
+		(property "Reference" "C53"
+			(at 71.755 50.165 0)
+			(effects
+				(font
+					(size 1.27 1.27)
+				)
+				(justify left)
+			)
+		)
+		(property "Value" "1.0uF"
+			(at 71.12 54.61 0)
+			(effects
+				(font
+					(size 1.27 1.27)
+				)
+				(justify left)
+			)
+		)
+		(property "Footprint" "Capacitor_SMD:C_0402_1005Metric"
+			(at 71.12 52.07 0)
+			(effects
+				(font
+					(size 1.27 1.27)
+				)
+				(hide yes)
+			)
+		)
+		(property "Datasheet" "~"
+			(at 71.12 52.07 0)
+			(effects
+				(font
+					(size 1.27 1.27)
+				)
+				(hide yes)
+			)
+		)
+		(property "Description" ""
+			(at 71.12 52.07 0)
+			(effects
+				(font
+					(size 1.27 1.27)
+				)
+				(hide yes)
+			)
+		)
+		(pin "1"
+		)
+		(pin "2"
+		)
+		(instances
+			(project "usb3-gmm7550"
+				(path "/e63e39d7-6ac0-4ffd-8aa3-1841a4541b55/60a01b67-a296-4e5c-ae04-350714992f76"
+					(reference "C53")
+					(unit 1)
+				)

Commit message: Final touches -- revision 1.0 schematic is released
Parts:
- U21: value 74LVC1G06 -> SN74LVC1G06DBV
Changed lines of the file:
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@@
 	(title_block
 		(title "GMM-7550 USB3 Adapter")
-		(date "2025-10-01")
-		(rev "0.9.5")
+		(date "2025-10-10")
+		(rev "1.0")
 	)
 	(text "Amber"
@@
 			)
 		)
-		(property "Value" "74LVC1G06"
-			(at 186.69 128.27 0)
+		(property "Value" "SN74LVC1G06DBV"
+			(at 189.23 128.27 0)
 			(effects
 				(font
