File: usb3-gmm7550.kicad/usb3.kicad_sch (KiCad schematic)
At the start: 31 parts, among them J1 USB_C_Receptacle, U1 ECMF4-40A100N10, U2 ECMF4-40A100N10, U3 ECMF02-2AMX6, U4 AP7330, U5 TUSB542

Commit message: Final touches -- revision 1.0 schematic is released
Parts:
- D2: value PESD752DCKR -> ESD752DCKR
- U4: value AP7330 -> AP7330D
Changed lines of the file:
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@@
 	(title_block
 		(title "GMM-7550 USB3 Adapter")
-		(date "2025-10-01")
-		(rev "0.9.5")
+		(date "2025-10-10")
+		(rev "1.0")
 	)
 	(text "Copyright (c) 2025 Anton Kuzmin <ak@gmm7550.dev>\n\nThis documentation is distributed under the terms of\nthe CERN-OHL-P v2 (https://cern.ch/cern-ohl).\n\nThis project was funded through the NGI0 Common Fund,\na fund established by NLnet foundation."
@@
 			)
 		)
-		(property "Value" "PESD752DCKR"
+		(property "Value" "ESD752DCKR"
 			(at 107.95 31.7499 90)
 			(effects
@@
 			)
 		)
-		(property "Value" "AP7330"
+		(property "Value" "AP7330D"
 			(at 101.6 154.94 0)
 			(effects
